File: designs/tc6/tc6.sch (KiCad schematic (older format))
At the start: 19 parts, among them J1001 SSM-104-L-SV, P1 TC2030, U1001 MCP6001-OT

Commit message: migrating to version6
Parts:
- BRD1: footprint tc5:DemoBoard -> tc6:DemoBoard
- J1001: symbol tc5-rescue:Conn_01x04_Male-Connector -> tc6-rescue:Conn_01x04_Male-Connector
- P1: footprint tc5:TC2030-MCP-FP -> tc6:TC2030-MCP-FP
- QR1: footprint tc5:TC5 -> tc6:TC5; symbol tc5-rescue:SYM_Arrow_Normal-Graphic -> tc6-rescue:SYM_Arrow_Normal-Graphic
- R1001: symbol tc5-rescue:R_Small-Device -> tc6-rescue:R_Small-Device
- TP1001, TP1002, TP1003, TP1004, TP1005, TP1006: symbol tc5-rescue:TestPoint_Probe-Connector -> tc6-rescue:TestPoint_Probe-Connector
- U1001: symbol tc5-rescue:MCP6001-OT-Amplifier_Operational -> tc6-rescue:MCP6001-OT-Amplifier_Operational
Changed lines of the file:
@@
 $EndDescr
 $Comp
-L tc5-rescue:SYM_Arrow_Normal-Graphic QR1
+L tc6-rescue:SYM_Arrow_Normal-Graphic QR1
 U 1 1 61C5D077
 P 1925 1450
 F 0 "QR1" H 1925 1510 50  0001 C CNN
 F 1 "Product QR Code" H 1935 1400 50  0001 C CNN
-F 2 "tc5:TC5" H 1925 1450 50  0001 C CNN
+F 2 "tc6:TC5" H 1925 1450 50  0001 C CNN
 F 3 "~" H 1925 1450 50  0001 C CNN
 F 4 "virtual" H 1925 1450 50  0001 C CNN "manf"
@@
 Symbol to represent QRCode on PCB
 $Comp
-L tc5-rescue:MCP6001-OT-Amplifier_Operational U1001
+L tc6-rescue:MCP6001-OT-Amplifier_Operational U1001
 U 1 1 61C5DBDB
 P 3300 2375
@@
 $EndComp
 $Comp
-L tc5-rescue:R_Small-Device R1001
+L tc6-rescue:R_Small-Device R1001
 U 1 1 61C60726
 P 3225 3100
@@
 Connection ~ 3600 3100
 $Comp
-L tc5-rescue:Conn_01x04_Male-Connector J1001
+L tc6-rescue:Conn_01x04_Male-Connector J1001
 U 1 1 61C635DD
 P 1525 2250
@@
 	1725 2450 1950 2450
 $Comp
-L tc5-rescue:VCC-power #PWR0101
+L tc6-rescue:VCC-power #PWR0101
 U 1 1 61C66B30
 P 1950 2150
@@
 $EndComp
 $Comp
-L tc5-rescue:GND-power #PWR0102
+L tc6-rescue:GND-power #PWR0102
 U 1 1 61C67A4F
 P 1950 2250
@@
 $EndComp
 $Comp
-L tc5-rescue:VCC-power #PWR0103
+L tc6-rescue:VCC-power #PWR0103
 U 1 1 61C686E2
 P 3200 2075
@@
 $EndComp
 $Comp
-L tc5-rescue:GND-power #PWR0104
+L tc6-rescue:GND-power #PWR0104
 U 1 1 61C68E55
 P 3200 2675
@@
 _AOPIN+
 $Comp
-L tc5-rescue:TestPoint_Probe-Connector TP1003
+L tc6-rescue:TestPoint_Probe-Connector TP1003
 U 1 1 61C6D8DC
 P 4100 3100
@@
 $EndComp
 $Comp
-L tc5-rescue:TestPoint_Probe-Connector TP1002
+L tc6-rescue:TestPoint_Probe-Connector TP1002
 U 1 1 61C6F0D8
 P 2875 3100
@@
 Connection ~ 2875 3100
 $Comp
-L tc5-rescue:TestPoint_Probe-Connector TP1001
+L tc6-rescue:TestPoint_Probe-Connector TP1001
 U 1 1 61C7065D
 P 2850 2275
@@
 $EndComp
 $Comp
-L tc5-rescue:TestPoint_Probe-Connector TP1005
+L tc6-rescue:TestPoint_Probe-Connector TP1005
 U 1 1 61C76041
 P 1925 3175
@@
 $EndComp
 $Comp
-L tc5-rescue:TestPoint_Probe-Connector TP1004
+L tc6-rescue:TestPoint_Probe-Connector TP1004
 U 1 1 61C77FC1
 P 1925 2950
@@
 $EndComp
 $Comp
-L tc5-rescue:GND-power #PWR0105
+L tc6-rescue:GND-power #PWR0105
 U 1 1 61C784ED
 P 1775 3175
@@
 	1775 3175 1925 3175
 $Comp
-L tc5-rescue:VCC-power #PWR0106
+L tc6-rescue:VCC-power #PWR0106
 U 1 1 61C78DD6
 P 1775 2950
@@
 F 0 "BRD1" H 2000 1165 50  0001 C CNN
 F 1 "SYM_Arrow_XLarge" H 2000 995 50  0001 C CNN
-F 2 "tc5:DemoBoard" H 2000 1075 50  0001 C CNN
+F 2 "tc6:DemoBoard" H 2000 1075 50  0001 C CNN
 F 3 "~" H 2000 1075 50  0001 C CNN
 	1    2000 1075
@@
 	3150 3700 3850 3700
 $Comp
-L tc5-rescue:VCC-power #PWR0107
+L tc6-rescue:VCC-power #PWR0107
 U 1 1 6242683E
 P 3450 3850
@@
 $EndComp
 $Comp
-L tc5-rescue:TestPoint_Probe-Connector TP1006
+L tc6-rescue:TestPoint_Probe-Connector TP1006
 U 1 1 62428AED
 P 3150 3700
@@
 $EndComp
 $Comp
-L tc5-rescue:VCC-power #PWR0108
+L tc6-rescue:VCC-power #PWR0108
 U 1 1 6242C310
 P 3650 4200
@@
 F 0 "P1" H 5025 1964 50  0000 C CNN
 F 1 "TC2030" H 5025 1875 50  0000 C CNN
-F 2 "tc5:TC2030-MCP-FP" H 4975 1650 50  0001 C CNN
+F 2 "tc6:TC2030-MCP-FP" H 4975 1650 50  0001 C CNN
 F 3 "~" H 4975 1650 50  0001 C CNN
 	1    4975 1650
