File: designs/tc7/tc7.kicad_sch (KiCad schematic)
At the start: 19 parts, among them J1001 SSM-104-L-SV, P1 TC2030, U1001 MCP6001-OT

Commit message: Demonstrate diff issue when PCB changes
Parts:
- BRD1: footprint tc7:DemoBoard -> tc7:biggerPCB
Changed lines of the file:
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@@
       (effects (font (size 1.27 1.27)) hide)
     )
-    (property "Footprint" "tc7:DemoBoard" (at 50.8 27.305 0)
+    (property "Footprint" "tc7:biggerPCB" (at 50.8 27.305 0)
       (effects (font (size 1.27 1.27)) hide)
     )

Commit message: Add test case regarding value
Parts:
- R1001: S1MN (none) -> Vishay; S1PN (none) -> CRCW060310K0FKEAHP; manf Dummy -> Vishay; manf# 10k -> CRCW060310K0FKEA
Changed lines of the file:
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@@
       (effects (font (size 1.27 1.27)) hide)
     )
-    (property "manf" "Dummy" (at 81.28 78.74 0)
+    (property "manf" "Vishay" (at 81.28 78.74 0)
       (effects (font (size 1.27 1.27)) hide)
     )
-    (property "manf#" "10k" (at 81.28 78.74 0)
+    (property "manf#" "CRCW060310K0FKEA" (at 81.28 78.74 0)
       (effects (font (size 1.27 1.27)) hide)
     )
@@
       (effects (font (size 1.27 1.27)) hide)
     )
+    (property "S1MN" "Vishay" (at 81.28 78.74 0)
+      (effects (font (size 1.27 1.27)) hide)
+    )
+    (property "S1PN" "CRCW060310K0FKEAHP" (at 81.28 78.74 0)
+      (effects (font (size 1.27 1.27)) hide)
+    )
+    (property "S1PL" "" (at 81.28 78.74 0)
+      (effects (font (size 1.27 1.27)) hide)
+    )
+    (property "S2MN" "" (at 81.28 78.74 0)
+      (effects (font (size 1.27 1.27)) hide)
+    )
+    (property "S2PN" "" (at 81.28 78.74 0)
+      (effects (font (size 1.27 1.27)) hide)
+    )
+    (property "S2PL" "" (at 81.28 78.74 0)
+      (effects (font (size 1.27 1.27)) hide)
+    )
+    (property "comment" "" (at 81.28 78.74 0)
+      (effects (font (size 1.27 1.27)) hide)
+    )
+    (property "desc" "" (at 81.28 78.74 0)
+      (effects (font (size 1.27 1.27)) hide)
+    )
